File: haradware/scl3300-evb.kicad_pcb (KiCad board)
At the start: 2 copper layers, 65 x 40 mm, 67 parts, among them J1 SMA, J2 STLINK, J3 BOOT1, J4 BOOT0, P1 USB_C_Receptacle_USB2.0_16P, SW1 RESET, SW2 SAMPLERATE, SW3 OPTIONS, U1 NEO-M8M, U2 AMS1117-3.3, U3 AT24CS08-SSHM, U4 SCL3300-D01, U5 CH340N, U6 STM32F103C8Tx, U7 SSD1306, Y1 SG-8002CA 8M-PCML0

Commit message: fix: SCL3300-D01 footprint
Parts:
- U4: footprint evb:SCL3300-D01 -> evb:DFL-12_L8.6-W7.0-P1.00-LS7.6-BL
- moved U4 0.40 mm to (104.3, 105.0), turned to -90 degrees
- moved C8 0.06 mm to (105.7, 99.3)
- turned D3 to 0 degrees
Connections:
- D3 pad 1: /+5V -> Net-(D2-A)
Routing:
- net Net-(D2-A): track 19.5 -> 23.3 mm
- net /+5V: track 18.6 -> 14.8 mm
- net Net-(BT1-+): track 39.0 -> 37.8 mm
- net /+3V3: track 228.1 -> 227.0 mm
- net /GNSS_RESET: track 31.8 -> 31.1 mm
- net /MCU_SCLK: track 31.6 -> 32.2 mm
- net GND: vias 76 -> 77
Other:
- board text added: "REV.20260705"
- board text removed: "BOOT0"
- board text removed: "BOOT1"
- board text removed: "REV.20251015"
