File: haradware/scl3300-evb.kicad_sch (KiCad schematic)
At the start: 67 parts, among them J1 SMA, J2 STLINK, J3 BOOT1, J4 BOOT0, P1 USB_C_Receptacle_USB2.0_16P, SW1 RESET, SW2 SAMPLERATE, SW3 OPTIONS, U1 NEO-M8M, U2 AMS1117-3.3, U3 AT24CS08-SSHM, U4 SCL3300-D01, U5 CH340N, U6 STM32F103C8Tx, U7 SSD1306, Y1 SG-8002CA 8M-PCML0

Commit message: fix: SCL3300-D01 footprint
Parts:
- U4: footprint evb:SCL3300-D01 -> evb:DFL-12_L8.6-W7.0-P1.00-LS7.6-BL
- U7: footprint Connector_PinSocket_2.54mm:PinSocket_1x04_P2.54mm_Vertical -> Explorer:SSD1306
Connections:
- net GND: now also P1.SH (SHIELD); no longer P1.S1 (SHIELD)
Changed lines of the file:
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@@
 			)
 		)
+		(property "Sim.Pins" "1=K 2=A"
+			(at 127 180.34 0)
+			(hide yes)
+			(show_name no)
+			(do_not_autoplace no)
+			(effects
+				(font
+					(size 1.27 1.27)
+				)
+			)
+		)
 		(pin "2"
 		)
@@
 			)
 		)
+		(property "Sim.Pins" "1=K 2=A"
+			(at 153.67 67.31 0)
+			(hide yes)
+			(show_name no)
+			(do_not_autoplace no)
+			(effects
+				(font
+					(size 1.27 1.27)
+				)
+			)
+		)
 		(pin "1"
 		)
@@
 			)
 		)
-		(property "Footprint" "Connector_PinSocket_2.54mm:PinSocket_1x04_P2.54mm_Vertical"
+		(property "Footprint" "Explorer:SSD1306"
 			(at 264.16 85.09 0)
 			(hide yes)
@@
 			)
 		)
-		(property "Footprint" "evb:SCL3300-D01"
+		(property "Footprint" "evb:DFL-12_L8.6-W7.0-P1.00-LS7.6-BL"
 			(at 134.62 127 0)
 			(hide yes)
@@
 			)
 		)
+		(property "Sim.Pins" "1=K 2=A"
+			(at 153.67 76.2 0)
+			(hide yes)
+			(show_name no)
+			(do_not_autoplace no)
+			(effects
+				(font
+					(size 1.27 1.27)
+				)
+			)
+		)
 		(pin "1"
 		)
@@
 		(pin "A8"
 		)
-		(pin "S1"
+		(pin "SH"
 		)
 		(pin "A4"
@@
 			)
 		)
+		(property "Sim.Device" "V"
+			(at 59.69 26.67 0)
+			(hide yes)
+			(show_name no)
+			(do_not_autoplace no)
+			(effects
+				(font
+					(size 1.27 1.27)
+				)
+			)
+		)
+		(property "Sim.Type" "DC"
+			(at 59.69 26.67 0)
+			(hide yes)
+			(show_name no)
+			(do_not_autoplace no)
+			(effects
+				(font
+					(size 1.27 1.27)
+				)
+			)
+		)
+		(property "Sim.Pins" "1=+ 2=-"
+			(at 59.69 26.67 0)
+			(hide yes)
+			(show_name no)
+			(do_not_autoplace no)
+			(effects
+				(font
+					(size 1.27 1.27)
+				)
+			)
+		)
 		(pin "2"
 		)
@@
 			(at 153.67 58.42 0)
 			(hide yes)
+			(show_name no)
+			(do_not_autoplace no)
+			(effects
+				(font
+					(size 1.27 1.27)
+				)
+			)
+		)
+		(property "Sim.Pins" "1=K 2=A"
+			(at 153.67 58.42 0)
+			(hide yes)
